Commit message: work with arduino

File: install/manipulator_description/share/manipulator_description/urdf/manipulator.urdf.xacro (robot description, xacro)
@@ -125,5 +125,5 @@
         <axis xyz="0 0 1"/>
         <!-- Reasonable limits (modify as needed) -->
-        <limit lower="-3.14" upper="3.14" effort="2.0" velocity="5.0"/>
+        <limit lower="-1.57" upper="1.57" effort="2.0" velocity="5.0"/>
     </joint>
     <link name="h_arm">
@@ -157,5 +157,5 @@
         <!-- Rotation around X-axis -->
         <axis xyz="1 0 0"/>
-        <limit lower="-1.57" upper="1.57" effort="2.0" velocity="3.0"/>
+        <limit lower="-0.79" upper="1.57" effort="2.0" velocity="3.0"/>
     </joint>
     <link name="motor_3">
@@ -188,5 +188,5 @@
         <!-- Rotation around X-axis -->
         <axis xyz="1 0 0"/>
-        <limit lower="-1.57" upper="1.57" effort="2.0" velocity="3.0"/>
+        <limit lower="-0.79" upper="0.79" effort="2.0" velocity="3.0"/>
     </joint>
     <link name="rod">
@@ -311,5 +311,5 @@
         <!-- Rotation about Y-axis -->
         <axis xyz="0 1 0"/>
-        <limit lower="0" upper="1.2" effort="1.0" velocity="2.0"/>
+        <limit lower="0" upper="0.79" effort="1.0" velocity="2.0"/>
     </joint>
     <link name="gripper_R">
@@ -345,5 +345,5 @@
         <!-- Rotation about Y-axis -->
         <axis xyz="0 1 0"/>
-        <limit lower="-1.2" upper="0" effort="1.0" velocity="2.0"/>
+        <limit lower="-0.79" upper="0" effort="1.0" velocity="2.0"/>
         <mimic joint="joint_4" multiplier="-1"/>
     </joint>

File: install/manipulator_description/share/manipulator_description/urdf/manipulator_ros2_control.xacro (robot description, xacro)
@@ -31,6 +31,6 @@
         <joint name="joint_1">
             <command_interface name="position">
-                <param name="min">-3.14159265359</param>
-                <param name="max">3.14159265359</param>
+                <param name="min">-1.57</param>
+                <param name="max">1.57</param>
             </command_interface>
             <state_interface name="position"/>
@@ -39,6 +39,6 @@
         <joint name="joint_2">
             <command_interface name="position">
-                <param name="min">-1.57079632679</param>
-                <param name="max">1.57079632679</param>
+                <param name="min">-0.79</param>
+                <param name="max">1.57</param>
             </command_interface>
             <state_interface name="position"/>
@@ -47,6 +47,6 @@
         <joint name="joint_3">
             <command_interface name="position">
-                <param name="min">-1.57079632679</param>
-                <param name="max">1.57079632679</param>
+                <param name="min">-0.79</param>
+                <param name="max">0.79</param>
             </command_interface>
             <state_interface name="position"/>
@@ -56,5 +56,5 @@
             <command_interface name="position">
                 <param name="min">0.0</param>
-                <param name="max">1.2</param>
+                <param name="max">0.79</param>
             </command_interface>
             <state_interface name="position"/>
