Commit message: with pc

File: install/manipulator_description/share/manipulator_description/urdf/manipulator_ros2_control.xacro (robot description, xacro)
@@ -29,5 +29,4 @@
                 <param name="baudrate">1000000</param>  <!--serial speed for the bus (1Mbps for STS3215)-->
                 <param name="servo_ids">1,2,3</param>
-                <param name="gpio_gripper">22</param>
                 <!-- STS3215 register map (override if your firmware differs) -->
                 <param name="goal_position_addr">0x2A</param> <!-- register address to write a target position. -->
@@ -41,5 +40,5 @@
                 <!-- Default STS3215 motion profile -->
                 <param name="servo_speed">1500</param>
-                <param name="servo_acceleration">100</param>
+                <param name="servo_acceleration">30</param>
                 <!-- STS3215 tuning defaults -->
                 <param name="tuning_enable">true</param>
@@ -51,16 +50,28 @@
                 <param name="punch">16</param>
                 <!-- Per-servo tuning overrides (indexed by joint order 1..N) -->
-                <param name="position_p_gain_1">36</param>
-                <param name="position_d_gain_1">36</param>
+                <param name="position_p_gain_1">20</param>
+                <param name="position_d_gain_1">60</param>
                 <param name="position_i_gain_1">2</param>
-                <param name="velocity_p_gain_1">20</param>
-                <param name="velocity_i_gain_1">50</param>
-                <param name="position_p_gain_2">28</param>
-                <param name="position_d_gain_2">30</param>
-                <param name="position_i_gain_2">4</param>
-                <param name="position_p_gain_3">32</param>
-                <param name="position_d_gain_3">24</param>
-                <param name="deadband_cw_1">2</param>
-                <param name="deadband_ccw_1">2</param>
+                <param name="velocity_p_gain_1">10</param>
+                <param name="velocity_i_gain_1">200</param>
+                <param name="position_p_gain_2">25</param>
+                <param name="position_d_gain_2">50</param>
+                <param name="position_i_gain_2">10</param>
+                <param name="velocity_p_gain_2">10</param>
+                <param name="velocity_i_gain_2">200</param>
+                <param name="position_p_gain_3">30</param>
+                <param name="position_d_gain_3">45</param>
+                <param name="position_i_gain_3">6</param>
+                <param name="velocity_p_gain_3">10</param>
+                <param name="velocity_i_gain_3">200</param>
+                <param name="deadband_cw_1">6</param>
+                <param name="deadband_ccw_1">4</param>
+                <param name="deadband_cw_2">4</param>
+                <param name="deadband_ccw_2">4</param>
+                <param name="deadband_cw_3">4</param>
+                <param name="deadband_ccw_3">4</param>
+                <param name="punch_1">12</param>
+                <param name="punch_2">16</param>
+                <param name="punch_3">12</param>
                 <!-- Set true when firmware publishes measured servo position feedback -->
                 <param name="feedback_from_hardware">true</param>
@@ -91,12 +102,4 @@
             <state_interface name="position"/>
         </joint>
-        <!-- joint_4 (gripper_L) : URDF limits [0, 1.2] -->
-        <joint name="joint_4">
-            <command_interface name="position">
-                <param name="min">0.0</param>
-                <param name="max">0.79</param>
-            </command_interface>
-            <state_interface name="position"/>
-        </joint>
     </ros2_control>
 </robot>

Commit message: add velocity interface

File: install/manipulator_description/share/manipulator_description/urdf/manipulator_ros2_control.xacro (robot description, xacro)
@@ -37,9 +37,9 @@
                 <param name="position_raw_max">4095</param>
                 <!-- Servo angle range that maps to raw min/max -->
-                <param name="position_rad_min">-1.57</param>
-                <param name="position_rad_max">1.57</param>
-                <!-- Default STS3215 motion profile -->
+                <param name="position_rad_min">-3.14159</param>
+                <param name="position_rad_max">3.14159</param>
+                 <!-- Default STS3215 motion profile -->
                 <param name="servo_speed">1500</param>
-                <param name="servo_acceleration">100</param>
+                <param name="servo_acceleration">30</param>
                 <!-- STS3215 tuning defaults -->
                 <param name="tuning_enable">true</param>
@@ -51,37 +51,51 @@
                 <param name="punch">16</param>
                 <!-- Per-servo tuning overrides (indexed by joint order 1..N) -->
-                <param name="position_p_gain_1">36</param>
-                <param name="position_d_gain_1">36</param>
+                <param name="position_p_gain_1">20</param>
+                <param name="position_d_gain_1">60</param>
                 <param name="position_i_gain_1">2</param>
-                <param name="velocity_p_gain_1">20</param>
-                <param name="velocity_i_gain_1">50</param>
-                <param name="position_p_gain_2">28</param>
-                <param name="position_d_gain_2">30</param>
-                <param name="position_i_gain_2">4</param>
-                <param name="position_p_gain_3">32</param>
-                <param name="position_d_gain_3">24</param>
-                <param name="deadband_cw_1">2</param>
-                <param name="deadband_ccw_1">2</param>
+                <param name="velocity_p_gain_1">10</param>
+                <param name="velocity_i_gain_1">200</param>
+                <param name="position_p_gain_2">25</param>
+                <param name="position_d_gain_2">50</param>
+                <param name="position_i_gain_2">10</param>
+                <param name="velocity_p_gain_2">10</param>
+                <param name="velocity_i_gain_2">200</param>
+                <param name="position_p_gain_3">30</param>
+                <param name="position_d_gain_3">45</param>
+                <param name="position_i_gain_3">6</param>
+                <param name="velocity_p_gain_3">10</param>
+                <param name="velocity_i_gain_3">200</param>
+                <param name="deadband_cw_1">6</param>
+                <param name="deadband_ccw_1">4</param>
+                <param name="deadband_cw_2">4</param>
+                <param name="deadband_ccw_2">4</param>
+                <param name="deadband_cw_3">4</param>
+                <param name="deadband_ccw_3">4</param>
+                <param name="punch_1">12</param>
+                <param name="punch_2">16</param>
+                <param name="punch_3">12</param>
                 <!-- Set true when firmware publishes measured servo position feedback -->
                 <param name="feedback_from_hardware">true</param>
             </hardware>
         </xacro:unless>
-        <!-- joint_1 (razor_connector -> motor_2) : URDF limits [-3.14, 3.14] -->
+        <!-- joint_1 (razor_connector -> motor_2) : URDF limits [-2.35619, 2.35619] -->
         <joint name="joint_1">
             <command_interface name="position">
-                <param name="min">-1.57</param>
+                <param name="min">-2.35619</param>
+                <param name="max">2.35619</param>
+            </command_interface>
+            <state_interface name="position"/>
+            <state_interface name="velocity"/>
+        </joint>
+        <!-- joint_2 (motor_2 -> h_arm_L) : URDF limits [0, 1.57] -->
+        <joint name="joint_2">
+            <command_interface name="position">
+                <param name="min">0</param>
                 <param name="max">1.57</param>
             </command_interface>
             <state_interface name="position"/>
+            <state_interface name="velocity"/>
         </joint>
-        <!-- joint_2 (motor_2 -> h_arm_L) : URDF limits [-1.57, 1.57] -->
-        <joint name="joint_2">
-            <command_interface name="position">
-                <param name="min">-0.79</param>
-                <param name="max">1.57</param>
-            </command_interface>
-            <state_interface name="position"/>
-        </joint>
-        <!-- joint_3 (h_arm -> motor_3) : URDF limits [-1.57, 1.57] -->
+        <!-- joint_3 (h_arm -> motor_3) : URDF limits [-0.79, 0.79] -->
         <joint name="joint_3">
             <command_interface name="position">
@@ -90,6 +104,7 @@
             </command_interface>
             <state_interface name="position"/>
+            <state_interface name="velocity"/>
         </joint>
-        <!-- joint_4 (gripper_L) : URDF limits [0, 1.2] -->
+        <!-- joint_4 (gripper_L) : URDF limits [0, 0.79] -->
         <joint name="joint_4">
             <command_interface name="position">

File: src/manipulator_description/urdf/manipulator_ros2_control.xacro (robot description, xacro)
@@ -37,6 +37,6 @@
                 <param name="position_raw_max">4095</param>
                 <!-- Servo angle range that maps to raw min/max -->
-                <param name="position_rad_min">-1.57</param>
-                <param name="position_rad_max">1.57</param>
+                <param name="position_rad_min">-3.14159</param>
+                <param name="position_rad_max">3.14159</param>
                  <!-- Default STS3215 motion profile -->
                 <param name="servo_speed">1500</param>
@@ -79,21 +79,23 @@
             </hardware>
         </xacro:unless>
-        <!-- joint_1 (razor_connector -> motor_2) : URDF limits [-3.14, 3.14] -->
+        <!-- joint_1 (razor_connector -> motor_2) : URDF limits [-2.35619, 2.35619] -->
         <joint name="joint_1">
             <command_interface name="position">
-                <param name="min">-1.57</param>
+                <param name="min">-2.35619</param>
+                <param name="max">2.35619</param>
+            </command_interface>
+            <state_interface name="position"/>
+            <state_interface name="velocity"/>
+        </joint>
+        <!-- joint_2 (motor_2 -> h_arm_L) : URDF limits [0, 1.57] -->
+        <joint name="joint_2">
+            <command_interface name="position">
+                <param name="min">0</param>
                 <param name="max">1.57</param>
             </command_interface>
             <state_interface name="position"/>
+            <state_interface name="velocity"/>
         </joint>
-        <!-- joint_2 (motor_2 -> h_arm_L) : URDF limits [-1.57, 1.57] -->
-        <joint name="joint_2">
-            <command_interface name="position">
-                <param name="min">-0.79</param>
-                <param name="max">1.57</param>
-            </command_interface>
-            <state_interface name="position"/>
-        </joint>
-        <!-- joint_3 (h_arm -> motor_3) : URDF limits [-1.57, 1.57] -->
+        <!-- joint_3 (h_arm -> motor_3) : URDF limits [-0.79, 0.79] -->
         <joint name="joint_3">
             <command_interface name="position">
@@ -102,6 +104,7 @@
             </command_interface>
             <state_interface name="position"/>
+            <state_interface name="velocity"/>
         </joint>
-        <!-- joint_4 (gripper_L) : URDF limits [0, 1.2] -->
+        <!-- joint_4 (gripper_L) : URDF limits [0, 0.79] -->
         <joint name="joint_4">
             <command_interface name="position">
