Commit message: hardware_interface

File: src/manipulator_description/urdf/manipulator.urdf.xacro (robot description, xacro)
@@ -1,4 +1,6 @@
 <?xml version="1.0"?>
 <robot xmlns:xacro="http://www.ros.org/wiki/xacro" name="manipulator">
+    <xacro:arg name="is_sim" default="true"/>
+    <xacro:property name="is_sim" value="$(arg is_sim)"/>
     <xacro:include filename="$(find manipulator_description)/urdf/manipulator_gazebo.xacro"/>
     <xacro:include filename="$(find manipulator_description)/urdf/manipulator_ros2_control.xacro"/>

File: src/manipulator_description/urdf/manipulator_ros2_control.xacro (robot description, xacro)
@@ -11,7 +11,21 @@
     <!-- This <ros2_control> block configures the hardware/system plugin for ros2_control -->
     <ros2_control type="system" name="RobotSystem">
-        <hardware>
-            <plugin>gz_ros2_control/GazeboSimSystem</plugin>
-        </hardware>
+        <xacro:if value="${is_sim}">
+            <hardware>
+                <plugin>gz_ros2_control/GazeboSimSystem</plugin>
+            </hardware>
+            <!-- joint_5 mimics joint_4 with multiplier=-1 in the URDF -->
+            <joint name="joint_5">
+                <param name="mimic">joint_4</param>
+                <param name="multiplier">-1</param>
+                <state_interface name="position"/>
+            </joint>
+        </xacro:if>
+        <xacro:unless value="${is_sim}">
+            <hardware>
+                <plugin>manipulator_controller/ManipulatorInterface</plugin>
+                <param name="port">/dev/ttyACM0</param>
+            </hardware>
+        </xacro:unless>
         <!-- joint_1 (razor_connector -> motor_2) : URDF limits [-3.14, 3.14] -->
         <joint name="joint_1">
@@ -46,9 +60,4 @@
             <state_interface name="position"/>
         </joint>
-        <!-- joint_5 mimics joint_4 with multiplier=-1 in the URDF -->
-        <joint name="joint_5">
-            <param name="mimic">joint_4</param>
-            <param name="multiplier">-1</param>
-        </joint>
     </ros2_control>
 </robot>

Commit message: joint 3 inversed

File: src/manipulator_description/urdf/manipulator.urdf.xacro (robot description, xacro)
@@ -125,5 +125,5 @@
         <axis xyz="0 0 1"/>
         <!-- Reasonable limits (modify as needed) -->
-        <limit lower="-1.57" upper="1.57" effort="2.0" velocity="5.0"/>
+        <limit lower="-2.35619" upper="2.35619" effort="2.0" velocity="5.0"/>
     </joint>
     <link name="h_arm">
@@ -157,5 +157,5 @@
         <!-- Rotation around X-axis -->
         <axis xyz="1 0 0"/>
-        <limit lower="-0.79" upper="1.57" effort="2.0" velocity="3.0"/>
+        <limit lower="0" upper="1.57" effort="2.0" velocity="3.0"/>
     </joint>
     <link name="motor_3">

Commit message: now we can tune via code

File: src/manipulator_description/urdf/manipulator.urdf.xacro (robot description, xacro)
@@ -125,5 +125,5 @@
         <axis xyz="0 0 1"/>
         <!-- Reasonable limits (modify as needed) -->
-        <limit lower="-2.35619" upper="2.35619" effort="2.0" velocity="5.0"/>
+        <limit lower="-2.35619" upper="2.35619" effort="1.0" velocity="4.7"/>
     </joint>
     <link name="h_arm">
@@ -157,5 +157,5 @@
         <!-- Rotation around X-axis -->
         <axis xyz="1 0 0"/>
-        <limit lower="0" upper="1.57" effort="2.0" velocity="3.0"/>
+        <limit lower="0" upper="1.57" effort="1.0" velocity="3.0"/>
     </joint>
     <link name="motor_3">
@@ -188,5 +188,5 @@
         <!-- Rotation around X-axis -->
         <axis xyz="1 0 0"/>
-        <limit lower="-0.79" upper="0.79" effort="2.0" velocity="3.0"/>
+        <limit lower="-0.79" upper="0.79" effort="1.0" velocity="3.0"/>
     </joint>
     <link name="rod">
@@ -311,5 +311,5 @@
         <!-- Rotation about Y-axis -->
         <axis xyz="0 1 0"/>
-        <limit lower="0" upper="0.79" effort="1.0" velocity="2.0"/>
+        <limit lower="0" upper="0.79" effort="0.6" velocity="2.0"/>
     </joint>
     <link name="gripper_R">
@@ -345,5 +345,5 @@
         <!-- Rotation about Y-axis -->
         <axis xyz="0 1 0"/>
-        <limit lower="-0.79" upper="0" effort="1.0" velocity="2.0"/>
+        <limit lower="-0.79" upper="0" effort="0.6" velocity="2.0"/>
         <mimic joint="joint_4" multiplier="-1"/>
     </joint>

File: src/manipulator_description/urdf/manipulator_ros2_control.xacro (robot description, xacro)
@@ -42,4 +42,12 @@
                 <param name="servo_speed">1000</param>
                 <param name="servo_acceleration">50</param>
+                <!-- STS3215 tuning defaults -->
+                <param name="tuning_enable">true</param>
+                <param name="position_p_gain">32</param>
+                <param name="position_d_gain">32</param>
+                <param name="position_i_gain">0</param>
+                <param name="deadband_cw">1</param>
+                <param name="deadband_ccw">1</param>
+                <param name="punch">16</param>
                 <!-- Set true when firmware publishes measured servo position feedback -->
                 <param name="feedback_from_hardware">true</param>
